File: dabao_v3c.kicad_sch (KiCad schematic)
At the start: 48 parts, among them J1 USB_C_Receptacle_USB2.0_16P, SW1 SW_Push, SW2 SW_Push, U1 baochip1x, U3 Baochip, U4 MT3406, U5 EMS4000RSW, U6 MT3406, Y2 48.000MHz

Commit message: initial placement
Parts:
- removed SW1, SW2: SW_Push, common:SW_Push_1P1T_XKB_TS-1187A, symbol Switch:SW_Push
- added SW1, SW2: SKTAAAE010, xiao:SW4-SMD-2.8-2.6X1.6X0.53MM, symbol Seeed_libdb:Switch/311021459
- added TP11, TP12, TP16, TP7, TP8: Test Point, xiao:TP-1.6MM-ROUND, symbol Seeed_libdb:Misc/TP-1.6MM-ROUND
- added TP13, TP14, TP15: Test Point, Misc:TP-1.6MM-ROUND, symbol Seeed_libdb:Misc/TP-1.6MM-ROUND
- added U2: ~, xiao:MOUDLE14P-XIAO-HALF-HOLE, symbol Seeed_libadl:Module/XIAO-HALF-HOLE
- R11, R2, R5: footprint Resistor_SMD:R_0402_1005Metric -> Resistor_SMD:R_0201_0603Metric
- Y2: footprint Crystal:Crystal_SMD_3225-4Pin_3.2x2.5mm -> Crystal:Crystal_SMD_2016-4Pin_2.0x1.6mm; AltPN C70579 -> C2450980; LCSC C2892060 -> C2450980; VendorPN X322548MSB4SI -> ECS-480-8-47-JTN-TR
Connections:
- net GND: now also SW1.1 (A0), SW1.2 (A1), SW2.1 (A0), SW2.2 (A1), U2.13 (GND)
- net PC13: now also SW2.3 (B0), SW2.4 (B1)
- net VBUS: now also U2.14 (5V)
- net at R2.1: now also SW1.3 (B0), SW1.4 (B1)
- new net +3V3: U2.12 (3V3)
- new net GPIO0/D6/TX0: U2.7 (PB08_A6_D6_TX)
- new net GPIO10/D17/SPI1_SCK: TP11.1 (T)
- new net GPIO11/D15/SPI1_MOSI: TP7.1 (T)
- new net GPIO12/D16/SPI1_MISO: TP8.1 (T)
- new net GPIO16/D14/SDA0: TP13.1 (T)
- new net GPIO17/D13/SCL0: TP14.1 (T)
- new net GPIO1/D7/RX0: U2.8 (PB09_A7_D7_RX)
- new net GPIO20/D12/TX1: TP15.1 (T)
- new net GPIO21/D11/RX1: TP16.1 (T)
- new net GPIO26/D0/ADC0: U2.1 (PA02_A0_D0)
- new net GPIO27/D1/ADC1: U2.2 (PA4_A1_D1)
- new net GPIO28/D2/ADC2: U2.3 (PA10_A2_D2)
- new net GPIO2/D8/SPI0_SCK: U2.9 (PA7_A8_D8_SCK)
- new net GPIO3/D10/SPI0_MOSI: U2.11 (PA6_A10_D10_MOSI)
- new net GPIO4/D9/SPI0_MISO: U2.10 (PA5_A9_D9_MISO)
- new net GPIO5/D3/SPI0_CS: U2.4 (PA11_A3_D3)
- new net GPIO6/D4/SDA1: U2.5 (PA8_A4_D4_SDA)
- new net GPIO7/D5/SCL1: U2.6 (PA9_A5_D5_SCL)
- new net GPIO9/D18/SPI1_CS: TP12.1 (T)

Commit message: some bunnie edits, battery charging added
Parts:
- removed C12, C14, C16, C17: 10uF, 25V, X5R, Capacitor_SMD:C_0603_1608Metric, symbol common:root_3_Cap Semi
- removed D1: 1N5819WS, Diode_SMD:D_SOD-323, symbol Diode:1N4148WS
- removed H1, H2, H3, H4: MountingHole, MountingHole:MountingHole_2.2mm_M2_DIN965, symbol Mechanical:MountingHole
- removed L1, L2: 2.2uH MGFL2012F2R2MT-LF, Inductor_SMD:L_0805_2012Metric, symbol Device:L_Iron_Small
- removed R1, R10: 10k, 1%, Resistor_SMD:R_0201_0603Metric, symbol power-altium-import:root_3_Res1
- removed R6, R8: 100k, 1%, Resistor_SMD:R_0201_0603Metric, symbol power-altium-import:root_3_Res1
- removed R7: 453k, 1%, Resistor_SMD:R_0201_0603Metric, symbol power-altium-import:root_3_Res1
- removed R9: 43.2k, 1%, Resistor_SMD:R_0201_0603Metric, symbol power-altium-import:root_3_Res1
- removed TP11, TP12, TP16, TP7, TP8: Test Point, xiao:TP-1.6MM-ROUND, symbol Seeed_libdb:Misc/TP-1.6MM-ROUND
- removed TP13, TP14, TP15: Test Point, Misc:TP-1.6MM-ROUND, symbol Seeed_libdb:Misc/TP-1.6MM-ROUND
- removed U3: Baochip, common:Dabao_Vendor_Substrate, symbol common:Dabao
- removed U4, U6: MT3406, Package_TO_SOT_SMD:SOT-23-5, symbol common:MT3406
- added C14, C17, C19, C21: 10uF, Capacitor_SMD:C_0201_0603Metric, symbol Seeed_libadl:Capacitors/302010053
- added C16, C20, C22: 100nF, Capacitor_SMD:C_0201_0603Metric, symbol Seeed_libadl:Capacitors/302010271
- added C26: 1nF, Capacitor_SMD:C_0201_0603Metric, symbol Seeed_libdb:Capacitors/302010389
- added C27, C3, C6: 1uF, Capacitor_SMD:C_0201_0603Metric, symbol Seeed_libdb:Capacitors/302010730
- added D2: LMBR4010BST5G, xiao:DFN1006-2L, symbol Seeed_libadl:Diode/304021082
- added D3: LNZ8F5V6T5G, xiao:DFN1006-2L, symbol Seeed_libadl:Diode/304021082
- added L1, L3: 0.47uH, xiao:L0603, symbol Seeed_libadl:Inductor/303011858
- added Q1: LP0404N3T5G, xiao:PMOS_1.0X0.6X0.35MM, symbol Seeed_libadl:Mosfet/305031466
- added Q2: LN237N3T5G, xiao:PMOS_1.0X0.6X0.35MM, symbol Seeed_libadl:Mosfet/305030000
- added R12: 150K, xiao:R0201, symbol Seeed_libdb:Resistors/RC0201FR-07150KL
- added R13, R14, R16: 470K, Resistor_SMD:R_0201_0603Metric, symbol Seeed_libdb:Resistors/301010764
- added R15: 249K, Resistor_SMD:R_0201_0603Metric, symbol Seeed_libadl:Resistors/301013554
- added R19: 2.2K, Resistor_SMD:R_0201_0603Metric, symbol Seeed_libadl:Resistors/301010753
- added R20: 100R, Resistor_SMD:R_0201_0603Metric, symbol Seeed_libadl:Resistors/301010524
- added R6: 12.1k, Resistor_SMD:R_0201_0603Metric, symbol Seeed_libadl:Resistors/301013554
- added TP10, TP9: Test Point, xiao:TP-80X40MIL, symbol Seeed_libdb:Misc/TP-80X40MIL
- added U3, U9: SMD IC PMIC;DCDC Buck-ADJ-1A,Vin 1.95V to 5.5V,Vo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, xiao:BGA6-0.35-0.745X10.95X0.4MM, symbol Seeed_libadl:Ic/310032702
- added U7: SGM40567-4.2XG/TR, xiao:WLCSP-0.4-0.92X1.16X0.4MM, symbol Seeed_libadl:Ic/310032697
- added U8: SX1801CCR, xiao:WLCSP4-0.4-0.77X0.77X0.33MM, symbol Seeed_libdb:Ic/SX1801CCR
- R3: footprint Resistor_SMD:R_0402_1005Metric -> Resistor_SMD:R_0201_0603Metric
Connections:
- net +3V3 is gone; now on net +3.3V: U2.12 (3V3)
- net GPIO0/D6/TX0 is gone; now on net PB14: U2.7 (PB08_A6_D6_TX)
- net GPIO1/D7/RX0 is gone; now on net PB13: U2.8 (PB09_A7_D7_RX)
- net GPIO26/D0/ADC0 is gone; now on net PB3: U2.1 (PA02_A0_D0)
- net GPIO27/D1/ADC1 is gone; now on net PB4: U2.2 (PA4_A1_D1)
- net GPIO28/D2/ADC2 is gone; now on net PB1: U2.3 (PA10_A2_D2)
- net GPIO2/D8/SPI0_SCK is gone; now on net PC0: U2.9 (PA7_A8_D8_SCK)
- net GPIO3/D10/SPI0_MOSI is gone; now on net PC1: U2.11 (PA6_A10_D10_MOSI)
- net GPIO4/D9/SPI0_MISO is gone; now on net PC2: U2.10 (PA5_A9_D9_MISO)
- net GPIO5/D3/SPI0_CS is gone; now on net PB2: U2.4 (PA11_A3_D3)
- net GPIO6/D4/SDA1 is gone; now on net PB12: U2.5 (PA8_A4_D4_SDA)
- net GPIO7/D5/SCL1 is gone; now on net PB11: U2.6 (PA9_A5_D5_SCL)
- net +3.3V: now also C16.1, C17.1, C20.1, C21.1, L1.2, L3.2, U3.A2 (VOS), U9.A2 (VOS)
- net GND: now also C14.2, C16.2, C17.2, C19.2, C20.2, C21.2, C22.2, C26.2, C27.2, C3.2, C6.2, Q2.2 (S), R12.1, R14.1, R15.1, R16.1, R19.1, R6.1, TP10.1 (T), U3.A1 (GND), U7.B1 (F), U7.C2 (GND), U8.B1 (GND), U9.A1 (GND)
- net VBUS: now also C22.1, C3.1, D2.1, D3.2, Q2.3 (D), R16.2, R20.1, U7.A2 (VIN)
- net VSYS: now also C14.1, C19.1, D2.2, Q1.2 (S), U3.B1 (VIN), U3.C2 (EN), U9.B1 (VIN), U9.C2 (EN)
- new net: Q1.1 (G), R20.2
- new net: L1.1, U3.B2 (SW)
- new net: R6.2, U3.C1 (MODE)
- new net: C27.1, R13.2, U8.A1 (VOUT)
- new net: L3.1, U9.B2 (SW)
- new net: R15.2, U9.C1 (MODE)
- new net: D3.1, Q2.1 (G), R19.2
- new net: R12.2, U7.C1 (IREF)
- new net GPIO19/D22/BAT_ADC_EN: U8.B2 (EN)
- new net GPIO29_ADC3: C26.1, R13.1, R14.2
- new net NCHG: U7.B2 (NCHG)
- new net VBAT: C6.1, Q1.3 (D), TP9.1 (T), U7.A1 (BAT), U8.A2 (VIN)
Other:
- note added: "ICharge=24000/150K=160mA"
- note removed: "Vout = 0.6 * (1 + Rtop/Rbot) 0.85 = 0.6 * (1 + Rtop / 100k) Rtop = 41.67k 42.2k -> 0.8532v 43.2k -> 0.8592v Trim slightly high to ensure SW > LDO default voltage over tolerance"
- note removed: "Vout = 0.6 * (1 + Rtop/Rbot) 3.3 = 0.6 * (1 + Rtop / 100k) Rtop = 450k 453k -> 3.318V"
- moved on the sheet: C1, C10, C11, C13, C15, C18, C2, C4, C5, C7, C8, C9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

Commit message: tentative bao layout
Parts:
- removed U2: ~, xiao:MOUDLE14P-XIAO-HALF-HOLE, symbol Seeed_libadl:Module/XIAO-HALF-HOLE
- added R7: 5.1K, Resistor_SMD:R_0201_0603Metric, symbol Seeed_libadl:Resistors/301010885
- added U4: XIAO-HALF-HOLE-23P, xiao:MOUDLE23P-XIAO-HALF-HOLE, symbol libdb:Module/XIAO-HALF-HOLE-23P
Connections:
- net +0.9V: now also C16.1, C17.1, L1.2, U1.G7 (PF5), U3.A2 (VOS); no longer U1.F6 (PA6)
- net +3.3V: now also U4.12 (VCC_3V3); no longer C16.1, C17.1, L1.2, U1.D7 (PA7), U3.A2 (VOS)
- net GND: now also U1.G5 (PF4), U4.13 (GND); no longer U1.C4 (PA5), U1.E3 (PC5), U1.E4 (PF1), U1.F3 (PA3), U1.F4 (PC6)
- net PB1: now also U4.22 (GPIO12_DVP_Y7/SPI_MISO1)
- net PB11: now also U4.6 (GPIO6_D5/A5/I2C_SCL)
- net PB12: now also U4.5 (GPIO5_D4/A4/I2C_SDA)
- net PB13: now also U4.8 (U0RXD_D7/RX)
- net PB14: now also U4.7 (U0TXD_D6/TX)
- net PB2: now also U4.23 (GPIO13_DVP_PCLK/SPI_SCK1)
- net PC0: now also U4.9 (GPIO7_D8/A8/SCK)
- net PC1: now also U4.11 (GPIO9_D10/A10/MOSI)
- net PC2: now also U4.10 (GPIO8_D9/A9/MISO)
- net PC7: now also U4.20 (GPIO10_XMCLK/ADC_BAT)
- net PC8: now also U4.19 (GPIO42_PDM_CLK/TX1)
- net PC9: now also U4.18 (GPIO41_PDM_DATA/RX1); no longer U1.G3 (PA4)
- net VBUS: now also R7.2, U4.14 (VBUS)
- net PA1: now reaches U1.F2 (PF8_PA1)
- net PA1: now also U4.17 (GPIO40_CAM_SDA/I2S_WS)
- net PA5: now reaches U1.B5 (PB6)
- net PA5: now also U1.C4 (PA5), U4.2 (GPIO2_D1/A1)
- net NCHG: no longer names the net of U7.B2 (NCHG)
- net NCHG: now also R7.1
- new net PA0: U4.21 (GPIO11_DVP_Y8/SPI_MOSI1)
- new net PA4: U1.G3 (PA4), U4.1 (GPIO1_D0/A0)
- new net PA6: U1.F6 (PA6), U4.3 (GPIO3_D2/A2)
- new net PA7: U1.D7 (PA7), U4.4 (GPIO4_D3/A3)
- new net PC5: U1.E3 (PC5), U4.16 (GPIO39_CAM_SCL/I2S_SCK)
- new net PC6: U1.F4 (PC6), U4.15 (GPIO38_DVP_VSYNC/I2S_SD)
Other:
- note removed: "ADC mux"

Commit message: now with more pins
Parts:
- removed TP1, TP2: TestPoint, TestPoint:TestPoint_Pad_D1.0mm, symbol Connector:TestPoint
- added TP1, TP2, TP3, TP4, TP5, TP6, TP7, TP8: TEST-POINT'4545', xiao:TP-D45MIL, symbol XIAO ESP32S3_v1.2_230725-eagle-import:TEST-POINT'4545'
Connections:
- net +3.3V: now also TP7.T
- net GND: now also TP8.T
- net PB3: now also TP6.T
- net PB4: now also TP5.T
- net PC10: now also TP2.T
- net PC11: now also TP1.T
- net USBCONN_N: now also TP3.T
- net USBCONN_P: now also TP4.T

Commit message: now with silk and logos and an led
Parts:
- added D1: WS2812B-1010, xiao:1010 RGB WS2812B, symbol LED:WS2812B-2020
Connections:
- net GND: now also D1.2 (VSS)
- net PC12: now also D1.3 (DIN)
- net VSYS: now also D1.4 (VDD)
- no-connect marks 21 -> 22
Changed lines of the file:
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@@
 	)
 	(no_connect
+		(at 143.51 213.36)
+	)
+	(no_connect
 		(at 300.99 91.44)
 	)
@@
 	(wire
 		(pts
+			(xy 121.92 213.36) (xy 128.27 213.36)
+		)
+		(stroke
+			(width 0)
+			(type default)
+		)
+	)
+	(wire
+		(pts
 			(xy 151.13 144.78) (xy 165.1 144.78)
 		)
@@
 	(wire
 		(pts
+			(xy 135.89 204.47) (xy 135.89 205.74)
+		)
+		(stroke
+			(width 0)
+			(type default)
+		)
+	)
+	(wire
+		(pts
 			(xy 217.17 248.92) (xy 217.17 252.73)
 		)
@@
 		)
 	)
+	(label "PC12"
+		(at 121.92 213.36 0)
+		(effects
+			(font
+				(size 1.27 1.27)
+			)
+			(justify left bottom)
+		)
+	)
 	(label "PC13"
 		(at 80.01 101.6 0)
@@
 	)
 	(symbol
+		(lib_id "P & G:GND")
+		(at 135.89 220.98 0)
+		(unit 1)
+		(exclude_from_sim no)
+		(in_bom yes)
+		(on_board yes)
+		(dnp no)
+		(property "Reference" "#PWR021"
+			(at 135.89 227.33 0)
+			(effects
+				(font
+					(size 1.27 1.27)
+				)
+				(hide yes)
+			)
+		)
+		(property "Value" "GND"
+			(at 135.89 224.79 0)
+			(effects
+				(font
+					(size 1.27 1.27)
+				)
+			)
+		)
+		(property "Footprint" ""
+			(at 135.89 220.98 0)
+			(effects
+				(font
+					(size 1.27 1.27)
+				)
+				(hide yes)
+			)
+		)
+		(property "Datasheet" ""
+			(at 135.89 220.98 0)
+			(effects
+				(font
+					(size 1.27 1.27)
+				)
+				(hide yes)
+			)
+		)
+		(property "Description" ""
+			(at 135.89 220.98 0)
+			(effects
+				(font
+					(size 1.27 1.27)
+				)
+				(hide yes)
+			)
+		)
+		(pin "1"
+		)
+		(instances
+			(project "dabao_v3c"
+				(path "/30b97054-956f-4926-8f71-e9554821c3b2"
+					(reference "#PWR021")
+					(unit 1)
+				)
+			)
+		)
+	)
+	(symbol
 		(lib_id "XIAO ESP32S3_v1.2_230725-eagle-import:TEST-POINT'4545'")
 		(at 205.74 215.9 0)
@@
 	)
 	(symbol
+		(lib_id "P & G:+5V")
+		(at 135.89 204.47 0)
+		(unit 1)
+		(exclude_from_sim no)
+		(in_bom yes)
+		(on_board yes)
+		(dnp no)
+		(property "Reference" "#PWR020"
+			(at 135.89 208.28 0)
+			(effects
+				(font
+					(size 1.27 1.27)
+				)
+				(hide yes)
+			)
+		)
+		(property "Value" "VSYS"
+			(at 135.636 200.406 0)
+			(effects
+				(font
+					(size 1.27 1.27)
+				)
+			)
+		)
+		(property "Footprint" ""
+			(at 135.89 204.47 0)
+			(effects
+				(font
+					(size 1.27 1.27)
+				)
+				(hide yes)
+			)
+		)
+		(property "Datasheet" ""
+			(at 135.89 204.47 0)
+			(effects
+				(font
+					(size 1.27 1.27)
+				)
+				(hide yes)
+			)
+		)
+		(property "Description" ""
+			(at 135.89 204.47 0)
+			(effects
+				(font
+					(size 1.27 1.27)
+				)
+				(hide yes)
+			)
+		)
+		(pin "1"
+		)
+		(instances
+			(project "dabao_v3c"
+				(path "/30b97054-956f-4926-8f71-e9554821c3b2"
+					(reference "#PWR020")
+					(unit 1)
+				)
+			)
+		)
+	)
+	(symbol
 		(lib_id "power-altium-import:P1.8V_BAR")
 		(at 346.71 198.12 180)
@@
 					(unit 1)
 				)
+			)
+		)
+	)
+	(symbol
+		(lib_id "LED:WS2812B-2020")
+		(at 135.89 213.36 0)
+		(unit 1)
+		(exclude_from_sim no)
+		(in_bom yes)
+		(on_board yes)
+		(dnp no)
+		(fields_autoplaced yes)
+		(property "Reference" "D1"
+			(at 149.86 206.9398 0)
+			(effects
+				(font
+					(size 1.27 1.27)
+				)
+			)
+		)
+		(property "Value" "WS2812B-1010"
+			(at 149.86 209.4798 0)
+			(effects
+				(font
+					(size 1.27 1.27)
+				)
+			)
+		)
+		(property "Footprint" "xiao:1010 RGB WS2812B"
+			(at 137.16 220.98 0)
+			(effects
+				(font
+					(size 1.27 1.27)
+				)
+				(justify left top)
+				(hide yes)
+			)
+		)
+		(property "Datasheet" "https://cdn-shop.adafruit.com/product-files/4684/4684_WS2812B-2020_V1.3_EN.pdf"
+			(at 138.43 222.885 0)
+			(effects
+				(font
+					(size 1.27 1.27)
+				)
+				(justify left top)
+				(hide yes)
+			)
+		)
+		(property "Description" "RGB LED with integrated controller, 2.0 x 2.0 mm, 12 mA"
+			(at 135.89 213.36 0)
+			(effects
+				(font
+					(size 1.27 1.27)
+				)
+				(hide yes)
+			)
+		)
+		(pin "1"
+		)
+		(pin "2"
+		)
+		(pin "3"
+		)
+		(pin "4"
+		)
+		(instances
+			(project "dabao_v3c"
+				(path "/30b97054-956f-4926-8f71-e9554821c3b2"
+					(reference "D1")
+					(unit 1)
+				)
