File: dabao_v3c.kicad_sch (KiCad schematic)
At the start: 73 parts, among them J1 USB_C_Receptacle_USB2.0_16P, Q1 LP0404N3T5G, Q2 LN237N3T5G, SW1 SKTAAAE010, SW2 SKTAAAE010, U1 baochip1x, U2 TPS22916CYFPR, U3 SMD IC PMIC;DCDC Buck-ADJ-1A,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, U4 XIAO-HALF-HOLE-23P, U5 SGM7222YWQ10/TR, U7 SGM40567-4.2XG/TR, U8 TPS22916CYFPR, U9 SMD IC PMIC;DCDC Buck-ADJ-1A,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, Y2 48.000MHz

Commit message: nearly final
Parts:
- D7, D8: footprint Diode:ESD-0201 -> xiao:ESD-0201
- R8: MYPN R-512-1P-1_16W-0402 -> (none)
Connections:
- net PC13 is gone; now on net PC13/BOOT: R8.2, U5.10 (SEL)
Changed lines of the file:
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@@
 	(wire
 		(pts
-			(xy 95.25 151.13) (xy 105.41 151.13)
+			(xy 95.25 151.13) (xy 107.95 151.13)
 		)
 		(stroke
@@
 		)
 	)
+	(label "PC13{slash}BOOT"
+		(at 107.95 151.13 180)
+		(effects
+			(font
+				(size 1.27 1.27)
+			)
+			(justify right bottom)
+		)
+	)
 	(label "PC2"
 		(at 218.44 60.96 180)
@@
 		)
 	)
-	(label "PC13"
-		(at 105.41 151.13 180)
-		(effects
-			(font
-				(size 1.27 1.27)
-			)
-			(justify right bottom)
-		)
-	)
 	(label "PC9"
 		(at 325.12 62.23 0)
@@
 			)
 		)
-		(property "Footprint" "Diode:ESD-0201"
+		(property "Footprint" "xiao:ESD-0201"
 			(at 63.5 102.87 0)
 			(effects
@@
 			)
 		)
-		(property "Footprint" "Diode:ESD-0201"
+		(property "Footprint" "xiao:ESD-0201"
 			(at 273.05 102.87 0)
 			(effects
@@
 			)
 		)
-		(property "MYPN" "R-512-1P-1_16W-0402"
+		(property "MYPN" ""
 			(at 94.742 145.542 0)
 			(effects

Commit message: nit pick fix
Parts:
- D7, D8: value DF2B7ASL,L3F -> B74121U0055M060; MPN DF2B7ASL,L3F -> B74121U0055M060; Manufacturer TOSHIBA -> TDK; SKU DF2B7ASL,L3F -> B74121U0055M060
- TP1, TP2, TP3, TP4, TP5, TP6, TP7, TP8: now left out of the parts list
